Commit message: fixed translations on joints and added camera mount stl

File: cobot_description/urdf/cobot_macro.urdf.xacro (robot description, xacro)
@@ -6,24 +6,6 @@
 <xacro:include filename="$(find cobot_description)/urdf/cobot.gazebo" />
 <link name="${prefix}base_link"/>
-<link name="${prefix}arm_link">
-  <inertial>
-    <origin xyz="0.09220015181506477 0.6335816505231302 0.03915806806155288" rpy="0 0 0"/>
-    <mass value="25.654256838266296"/>
-    <inertia ixx="0.336867" iyy="0.745441" izz="1.049342" ixy="-0.074207" iyz="-0.009932" ixz="-0.048262"/>
-  </inertial>
-  <visual>
-    <origin xyz="0 0 0" rpy="0 0 0"/>
-    <geometry>
-      <mesh filename="package://cobot_description/meshes/arm_link.stl" scale="0.001 0.001 0.001"/>
-    </geometry>
-    <material name="cobot_silver"/>
-  </visual>
-  <collision>
-    <origin xyz="0 0 0" rpy="0 0 0"/>
-    <geometry>
-      <mesh filename="package://cobot_description/meshes/arm_link.stl" scale="0.001 0.001 0.001"/>
-    </geometry>
-  </collision>
-</link>
+<!-- arm_link removed: was mocked Kinova arm from Fusion -->
+<!-- Real Kinova arm now mounts directly to tower_link -->
 <link name="${prefix}tower_link">
   <inertial>
@@ -146,36 +128,35 @@
   </collision>
 </link>
-<joint name="${prefix}Rigid 4" type="fixed">
-  <origin xyz="0.064742 -0.009761 -0.165019" rpy="1.570796 -1.570796 0.0"/>
-  <parent link="${prefix}tower_link"/>
-  <child link="${prefix}arm_link"/>
-</joint>
+<!-- Rigid 4 joint removed: connected tower_link to mocked arm_link -->
+<!-- Kinova arm now mounts directly to tower_link via kinova.urdf.xacro -->
+<!-- Original mount transform preserved below for reference: -->
+<!-- <origin xyz="0.064742 -0.009761 -0.165019" rpy="1.570796 -1.570796 0.0"/> -->
 <joint name="${prefix}Rigid 5" type="fixed">
-  <origin xyz="-0.0 -0.0 0.11" rpy="0.0 0.0 3.141593"/>
+  <origin xyz="0 0 0.110" rpy="0.0 0.0 3.141593"/>
   <parent link="${prefix}base_link"/>
   <child link="${prefix}tower_link"/>
 </joint>
 <joint name="${prefix}Rigid 9" type="fixed">
-  <origin xyz="-0.395 0.017 0.1612" rpy="0.0 -0.0 -3.141593"/>
+  <origin xyz="-0.3950 0.0170 0.27120" rpy="0.0 -0.0 -3.141593"/>
   <parent link="${prefix}tower_link"/>
   <child link="${prefix}camera_mount_link"/>
 </joint>
 <joint name="${prefix}Rigid 10" type="fixed">
-  <origin xyz="0.3823 0.002648 0.2897" rpy="-0.0 0.0 3.141593"/>
+  <origin xyz="-0.01270 0.019648 0.56090" rpy="-0.0 0.0 3.141593"/>
   <parent link="${prefix}camera_mount_link"/>
   <child link="${prefix}camera_bracket_15deg_link"/>
 </joint>
 <joint name="${prefix}Rigid 13" type="fixed">
-  <origin xyz="0.0007 0.061 0.1457" rpy="-0.0 -0.0 3.141593"/>
+  <origin xyz="0.00070 0.0610 0.25570" rpy="-0.0 -0.0 3.141593"/>
   <parent link="${prefix}tower_link"/>
   <child link="${prefix}touchscreen_mount_link"/>
 </joint>
 <joint name="${prefix}Rigid 14" type="fixed">
-  <origin xyz="0.143798 -0.082201 -0.121244" rpy="2.356194 -0.0 3.141593"/>
+  <origin xyz="0.144498 -0.021201 0.134456" rpy="2.356194 -0.0 3.141593"/>
   <parent link="${prefix}touchscreen_mount_link"/>
   <child link="${prefix}touchscreen_link"/>
 </joint>
 <joint name="${prefix}Rigid 16" type="fixed">
-  <origin xyz="0.0127 -0.081287 -0.541546" rpy="1.832596 -0.0 -0.0"/>
+  <origin xyz="0 -0.061639 0.019354" rpy="1.832596 -0.0 -0.0"/>
   <parent link="${prefix}camera_bracket_15deg_link"/>
   <child link="${prefix}kinect_link"/>

Commit message: add cobot base geometry

File: cobot_description/urdf/cobot_macro.urdf.xacro (robot description, xacro)
@@ -5,5 +5,24 @@
 <xacro:include filename="$(find cobot_description)/urdf/cobot.trans" />
 <xacro:include filename="$(find cobot_description)/urdf/cobot.gazebo" />
-<link name="${prefix}base_link"/>
+<link name="${prefix}base_link">
+  <inertial>
+    <origin xyz="0.004518 0.003782 -0.023908" rpy="0 0 0"/>
+    <mass value="317800"/>
+    <inertia ixx="6.196" iyy="8.576" izz="5.573" ixy="-0.2254" iyz="-0.05173" ixz="-0.002643"/>
+  </inertial>
+  <visual>
+    <origin xyz="0 0 0" rpy="0 0 0"/>
+    <geometry>
+      <mesh filename="package://cobot_description/meshes/base_link.stl" scale="0.001 0.001 0.001"/>
+    </geometry>
+    <material name="cobot_silver"/>
+  </visual>
+  <collision>
+    <origin xyz="0 0 0" rpy="0 0 0"/>
+    <geometry>
+      <mesh filename="package://cobot_description/meshes/base_link.stl" scale="0.001 0.001 0.001"/>
+    </geometry>
+  </collision>
+</link>
 <!-- arm_link removed: was mocked Kinova arm from Fusion -->
 <!-- Real Kinova arm now mounts directly to tower_link -->
