Commit message: fix world frame to cobot base_link

File: kortex_description/robots/gen3.xacro (robot description, xacro)
@@ -31,6 +31,12 @@
     <xacro:property name="initial_positions_file" default="$(arg initial_positions_file)"/>
     <link name="world" />
+    <link name="/cobot/base_link"/>
+    <joint name="world_to_cobot_base" type="fixed">
+        <parent link="world"/>
+        <child  link="/cobot/base_link"/>
+        <origin xyz="0 0 0" rpy="0 0 0"/>
+    </joint>
     <xacro:load_robot
-        parent="world"
+        parent="/cobot/base_link"
         arm="$(arg arm)"
         gripper="$(arg gripper)"
@@ -56,5 +62,5 @@
         use_external_cable="$(arg use_external_cable)"
         initial_positions="${xacro.load_yaml(initial_positions_file)}" >
-        <origin xyz="0 0 0" rpy="0 0 0" />  <!-- position robot in the world -->
+        <origin xyz="0 0 0.468" rpy="0 0 0" />  <!-- position robot in the world -->
     </xacro:load_robot>
     <xacro:cobot_collision/>

Commit message: add cobot urdf to kinova urdf

File: kortex_description/robots/gen3.xacro (robot description, xacro)
@@ -25,5 +25,5 @@
     <xacro:arg name="use_external_cable" default="false" />
     <xacro:include filename="$(find kortex_description)/robots/kortex_robot.xacro" />
-    <xacro:include filename="$(find kortex_description)/robots/cobot_collision.xacro"/>
+    <xacro:include filename="$(find cobot_description)/urdf/cobot_macro.urdf.xacro" />
     <!-- initial position for simulations (Mock Hardware, Gazebo, Ignition) -->
     <xacro:arg name="initial_positions_file" default="$(find kortex_description)/config/initial_positions.yaml"/>
@@ -31,12 +31,16 @@
     <xacro:property name="initial_positions_file" default="$(arg initial_positions_file)"/>
     <link name="world" />
-    <!-- <link name="cobot_base_link"/>
-    <joint name="world_to_cobot_base" type="fixed">
+    <!-- Instantiate real cobot with prefix -->
+    <xacro:cobot prefix="cobot_"/>
+    <!-- Connect cobot base to world -->
+    <joint name="world_to_cobot" type="fixed">
         <parent link="world"/>
-        <child  link="cobot_base_link"/>
+        <child link="cobot_base_link"/>
         <origin xyz="0 0 0" rpy="0 0 0"/>
-    </joint> -->
+    </joint>
+    <!-- Mount Kinova arm to cobot tower_link -->
+    <!-- Original mocked arm mount (Rigid 4): xyz="0.064742 -0.009761 -0.165019" rpy="1.570796 -1.570796 0.0" -->
     <xacro:load_robot
-        parent="world"
+        parent="cobot_tower_link"
         arm="$(arg arm)"
         gripper="$(arg gripper)"
@@ -62,6 +66,7 @@
         use_external_cable="$(arg use_external_cable)"
         initial_positions="${xacro.load_yaml(initial_positions_file)}" >
-        <origin xyz="0 0 0.468" rpy="0 0 0" />  <!-- position robot in the world -->
+        <!-- Origin: Kinova base_link mount position relative to cobot_tower_link -->
+        <!-- Adjusting Z to account for different base_link origin in real Kinova vs mocked arm -->
+        <origin xyz="-0.005362 -0.083288 0.32" rpy="0 0 0" />
     </xacro:load_robot>
-    <xacro:cobot_collision/>
 </robot>

File: kortex_description/robots/kinova.urdf.xacro (robot description, xacro)
@@ -33,6 +33,6 @@
   <!-- import main macro -->
   <xacro:include filename="$(find kortex_description)/robots/kortex_robot.xacro" />
-  <!-- ADD: include our collision macro -->
-  <xacro:include filename="$(find kortex_description)/robots/cobot_collision.xacro" />
+  <!-- ADD: include real cobot macro from cobot_description -->
+  <xacro:include filename="$(find cobot_description)/urdf/cobot_macro.urdf.xacro" />
   <!-- initial position for simulations (Mock Hardware, Gazebo, Ignition) -->
   <xacro:arg name="initial_positions_file" default="$(find kortex_description)/config/initial_positions.yaml"/>
@@ -41,6 +41,17 @@
   <!-- create link fixed to the "world" -->
   <link name="world" />
+  <!-- Instantiate real cobot with prefix -->
+  <xacro:cobot prefix="cobot_"/>
+  <!-- Connect cobot base to world -->
+  <joint name="world_to_cobot" type="fixed">
+    <parent link="world"/>
+    <child link="cobot_base_link"/>
+    <origin xyz="0 0 0" rpy="0 0 0"/>
+  </joint>
+  <!-- Mount Kinova arm to cobot tower_link -->
+  <!-- Transform from cobot_tower_link to Kinova base_link -->
+  <!-- Original mocked arm mount (Rigid 4): xyz="0.064742 -0.009761 -0.165019" rpy="1.570796 -1.570796 0.0" -->
   <xacro:load_robot
-    parent="world"
+    parent="cobot_tower_link"
     arm="$(arg arm)"
     gripper="$(arg gripper)"
@@ -66,7 +77,8 @@
     initial_positions="${xacro.load_yaml(initial_positions_file)}"
     moveit_active="$(arg moveit_active)">
-    <origin xyz="0 0 0" rpy="0 0 0" />  <!-- position robot in the world -->
+    <!-- Origin: Kinova base_link mount position relative to cobot_tower_link -->
+    <!-- Starting point uses old mocked arm position - measure actual mount in Fusion -->
+    <origin xyz="0.064742 -0.009761 -0.165019" rpy="1.570796 -1.570796 0.0" />
   </xacro:load_robot>
-  <xacro:cobot_collision/>
   <xacro:if value="$(arg sim_gazebo)">
     <!-- Gazebo plugins -->

Commit message: Fix positioning of kinova urdf relative to tower

File: kortex_description/robots/gen3.xacro (robot description, xacro)
@@ -67,6 +67,6 @@
         initial_positions="${xacro.load_yaml(initial_positions_file)}" >
         <!-- Origin: Kinova base_link mount position relative to cobot_tower_link -->
-        <!-- Adjusting Z to account for different base_link origin in real Kinova vs mocked arm -->
-        <origin xyz="-0.005362 -0.083288 0.32" rpy="0 0 0" />
+        <!-- Final measured values: 331mm above tower, rotated -90° (yaw) -->
+        <origin xyz="0 0 0.331" rpy="0 0 -1.571" />
     </xacro:load_robot>
 </robot>

File: kortex_description/robots/kinova.urdf.xacro (robot description, xacro)
@@ -78,6 +78,6 @@
     moveit_active="$(arg moveit_active)">
     <!-- Origin: Kinova base_link mount position relative to cobot_tower_link -->
-    <!-- Starting point uses old mocked arm position - measure actual mount in Fusion -->
-    <origin xyz="0.064742 -0.009761 -0.165019" rpy="1.570796 -1.570796 0.0" />
+    <!-- Final measured values: 331mm above tower, rotated -90° (yaw) -->
+    <origin xyz="0 0 0.331" rpy="0 0 -1.571" />
   </xacro:load_robot>
   <xacro:if value="$(arg sim_gazebo)">
