Commit message: fix base collision for moveit

File: kortex_description/robots/cobot_collision.xacro (robot description, xacro)
@@ -8,5 +8,5 @@
       base_height:=0.162
       tower_size:='0.125 0.125 0.306'
-      tower_xyz:='0 0 -0.306'">
+      tower_xyz:='0 0 -0.154'">
     <!-- BOX: chassis shell (collision only) -->
     <link name="cobot_base">
@@ -22,9 +22,8 @@
       <parent link="${mount_link}"/>
       <child  link="cobot_base"/>
-      <origin xyz="0 0 0" rpy="0 0 0"/>
     </joint>
     <link name="cobot_tower">
       <collision>
-        <origin xyz="0 0 ${base_height}" rpy="0 0 0"/>
+        <origin xyz="${tower_xyz}" rpy="0 0 0"/>
         <geometry>
           <box size="${tower_size}"/>
@@ -35,5 +34,4 @@
       <parent link="cobot_base"/>
       <child  link="cobot_tower"/>
-      <origin xyz="${tower_xyz}" rpy="0 0 0"/>
     </joint>
   </xacro:macro>

File: kortex_description/robots/gen3.xacro (robot description, xacro)
@@ -25,4 +25,5 @@
     <xacro:arg name="use_external_cable" default="false" />
     <xacro:include filename="$(find kortex_description)/robots/kortex_robot.xacro" />
+    <xacro:include filename="$(find kortex_description)/robots/cobot_collision.xacro"/>
     <!-- initial position for simulations (Mock Hardware, Gazebo, Ignition) -->
     <xacro:arg name="initial_positions_file" default="$(find kortex_description)/config/initial_positions.yaml"/>
@@ -57,3 +58,4 @@
         <origin xyz="0 0 0" rpy="0 0 0" />  <!-- position robot in the world -->
     </xacro:load_robot>
+    <xacro:cobot_collision/>
 </robot>

Commit message: fix base collision for moveit
update meshes; add touchscreen

add full body collision for cobot in kortex_description

finish full body self-collision checking with moveit

fix race condition in kinova_gen3_7dof_robotiq_2f_85_moveit_config/launch/robot.launch.py

fix world frame to cobot base_link

need kinect to arm base calibration

fix moveit

Fixing intermittent launching issues

back up at 1009

get arm working

File: kortex_description/robots/cobot_collision.xacro (robot description, xacro)
@@ -1,4 +1,7 @@
 <?xml version="1.0"?>
 <robot xmlns:xacro="http://www.ros.org/wiki/xacro" name="cobot_collision">
+  <material name="cobot_silver">
+    <color rgba="0.700 0.700 0.700 1.000"/>
+  </material>
   <!-- Parameters you can tweak at instantiation -->
   <xacro:macro name="cobot_collision" params="
@@ -8,6 +11,16 @@
       base_height:=0.162
       tower_size:='0.125 0.125 0.306'
-      tower_xyz:='0 0 -0.306'">
-    <!-- BOX: chassis shell (collision only) -->
+      tower_xyz:='0 0 -0.154'
+      touchscreen_mount_xyz:='-0.065 0 -0.07'
+      touchscreen_xyz:='-0.086 0.15 0.06'
+      touchscreen_rpy:='0.78 0 -1.5708'
+      supporter_460_size:='0.025 0.025 0.46'
+      supporter_460_xyz:='-0.0188 -0.168 -0.06'
+      supporter_580_size:='0.025 0.025 0.58'
+      supporter_580_xyz:='-0.0188 -0.387 0.24'
+      camera_bracket_xyz:='0.001 -0.387 0.497'
+      kinect_xyz:='0.06 -0.387 0.515'
+      kinect_rpy:='1.8326 0 1.5708'
+      ">
     <link name="cobot_base">
       <collision>
@@ -15,5 +28,4 @@
         <geometry>
             <cylinder radius="${base_radius}" length="${base_height}"/>
-          <!-- <box size="${box_size}"/> -->
         </geometry>
       </collision>
@@ -22,9 +34,8 @@
       <parent link="${mount_link}"/>
       <child  link="cobot_base"/>
-      <origin xyz="0 0 0" rpy="0 0 0"/>
     </joint>
     <link name="cobot_tower">
       <collision>
-        <origin xyz="0 0 ${base_height}" rpy="0 0 0"/>
+        <origin xyz="${tower_xyz}" rpy="0 0 0"/>
         <geometry>
           <box size="${tower_size}"/>
@@ -35,5 +46,90 @@
       <parent link="cobot_base"/>
       <child  link="cobot_tower"/>
-      <origin xyz="${tower_xyz}" rpy="0 0 0"/>
+    </joint>
+    <link name="touchscreen_mount">
+      <collision>
+        <origin xyz="${touchscreen_mount_xyz}" rpy="0 0 -1.5708"/>
+        <geometry>
+        <mesh filename="package://kortex_description/meshes/touchscreen_mount.stl" scale="0.001 0.001 0.001"/>
+        </geometry>
+      </collision>
+    </link>
+    <joint name="touchscreen_mount_fixed" type="fixed">
+      <parent link="cobot_tower"/>
+      <child  link="touchscreen_mount"/>
+    </joint>
+    <link name="touchscreen">
+      <collision>
+        <origin xyz="${touchscreen_xyz}" rpy="${touchscreen_rpy}"/>
+        <geometry>
+        <mesh filename="package://kortex_description/meshes/touchscreen.stl" scale="0.001 0.001 0.001"/>
+        </geometry>
+      </collision>
+    </link>
+    <joint name="touchscreen_fixed" type="fixed">
+      <parent link="touchscreen_mount"/>
+      <child  link="touchscreen"/>
+    </joint>
+    <link name="supporter_460">
+      <collision>
+        <origin xyz="${supporter_460_xyz}" rpy="1.5708 1.5708 0"/>
+        <geometry>
+          <box size="${supporter_460_size}"/>
+        </geometry>
+      </collision>
+    </link>
+    <joint name="supporter_460_fixed" type="fixed">
+      <parent link="cobot_tower"/>
+      <child  link="supporter_460"/>
+    </joint>
+    <link name="supporter_580">
+      <collision>
+        <origin xyz="${supporter_580_xyz}" rpy="0 0 0"/>
+        <geometry>
+          <box size="${supporter_580_size}"/>
+        </geometry>
+      </collision>
+    </link>
+    <joint name="supporter_580_fixed" type="fixed">
+      <parent link="cobot_tower"/>
+      <child  link="supporter_580"/>
+    </joint>
+    <link name="camera_bracket">
+      <collision>
+        <origin xyz="${camera_bracket_xyz}" rpy="0 0 1.5708"/>
+        <geometry>
+        <mesh filename="package://kortex_description/meshes/camera_bracket.stl" scale="0.001 0.001 0.001"/>
+        </geometry>
+      </collision>
+    </link>
+    <joint name="camera_bracket_fixed" type="fixed">
+      <parent link="cobot_tower"/>
+      <child  link="camera_bracket"/>
+    </joint>
+    <link name="kinect">
+      <collision>
+        <origin xyz="${kinect_xyz}" rpy="${kinect_rpy}"/>
+        <geometry>
+        <mesh filename="package://kortex_description/meshes/kinect.stl" scale="0.001 0.001 0.001"/>
+        </geometry>
+      </collision>
+    </link>
+    <joint name="kinect_fixed" type="fixed">
+      <parent link="camera_bracket"/>
+      <child  link="kinect"/>
+    </joint>
+    <link name="kinect_ablated">
+      <collision>
+        <origin xyz="${kinect_xyz}" rpy="${kinect_rpy}"/>
+        <geometry>
+          <!-- <box size="0.11 0.05 0.2"/> -->
+          <!-- alate 4cm -->
+          <box size="0.15 0.09 0.24"/>
+        </geometry>
+      </collision>
+    </link>
+    <joint name="kinect_ablated_fixed" type="fixed">
+      <parent link="camera_bracket"/>
+      <child  link="kinect_ablated"/>
     </joint>
   </xacro:macro>

File: kortex_description/robots/gen3.xacro (robot description, xacro)
@@ -24,9 +24,16 @@
     <xacro:arg name="use_external_cable" default="false" />
     <xacro:include filename="$(find kortex_description)/robots/kortex_robot.xacro" />
-    <!-- initial position for simulations (Mock Hardware, Gazebo) -->
+    <xacro:include filename="$(find kortex_description)/robots/cobot_collision.xacro"/>
+    <!-- initial position for simulations (Mock Hardware, Gazebo, Ignition) -->
     <xacro:arg name="initial_positions_file" default="$(find kortex_description)/config/initial_positions.yaml"/>
     <!-- convert to property to use substitution in function -->
     <xacro:property name="initial_positions_file" default="$(arg initial_positions_file)"/>
     <link name="world" />
+    <!-- <link name="cobot_base_link"/>
+    <joint name="world_to_cobot_base" type="fixed">
+        <parent link="world"/>
+        <child  link="cobot_base_link"/>
+        <origin xyz="0 0 0" rpy="0 0 0"/>
+    </joint> -->
     <xacro:load_robot
         parent="world"
@@ -53,5 +60,6 @@
         use_external_cable="$(arg use_external_cable)"
         initial_positions="${xacro.load_yaml(initial_positions_file)}" >
-        <origin xyz="0 0 0" rpy="0 0 0" />  <!-- position robot in the world -->
+        <origin xyz="0 0 0.468" rpy="0 0 0" />  <!-- position robot in the world -->
     </xacro:load_robot>
+    <xacro:cobot_collision/>
 </robot>

Commit message: update meshes; add touchscreen

File: kortex_description/robots/cobot_collision.xacro (robot description, xacro)
@@ -1,4 +1,7 @@
 <?xml version="1.0"?>
 <robot xmlns:xacro="http://www.ros.org/wiki/xacro" name="cobot_collision">
+  <material name="cobot_silver">
+    <color rgba="0.700 0.700 0.700 1.000"/>
+  </material>
   <!-- Parameters you can tweak at instantiation -->
   <xacro:macro name="cobot_collision" params="
@@ -8,6 +11,8 @@
       base_height:=0.162
       tower_size:='0.125 0.125 0.306'
-      tower_xyz:='0 0 -0.154'">
-    <!-- BOX: chassis shell (collision only) -->
+      tower_xyz:='0 0 -0.154'
+      touchscreen_mount_xyz:='0.0 -0.065 -0.07'
+      touchscreen_xyz:='-0.15 -0.086 0.06'
+      touchscreen_rpy:='0.78 0 0'">
     <link name="cobot_base">
       <collision>
@@ -15,5 +20,4 @@
         <geometry>
             <cylinder radius="${base_radius}" length="${base_height}"/>
-          <!-- <box size="${box_size}"/> -->
         </geometry>
       </collision>
@@ -35,4 +39,40 @@
       <child  link="cobot_tower"/>
     </joint>
+    <link name="touchscreen_mount">
+      <visual>
+        <origin xyz="${touchscreen_mount_xyz}" rpy="0 0 0"/>
+        <geometry>
+        <mesh filename="package://kortex_description/meshes/touchscreen_mount.stl" scale="0.001 0.001 0.001"/>
+        </geometry>
+      </visual>
+      <collision>
+        <origin xyz="${touchscreen_mount_xyz}" rpy="0 0 0"/>
+        <geometry>
+        <mesh filename="package://kortex_description/meshes/touchscreen_mount.stl" scale="0.001 0.001 0.001"/>
+        </geometry>
+      </collision>
+    </link>
+    <joint name="touchscreen_mount_fixed" type="fixed">
+      <parent link="cobot_tower"/>
+      <child  link="touchscreen_mount"/>
+    </joint>
+    <link name="touchscreen">
+      <visual>
+        <origin xyz="${touchscreen_xyz}" rpy="${touchscreen_rpy}"/>
+        <geometry>
+        <mesh filename="package://kortex_description/meshes/touchscreen.stl" scale="0.001 0.001 0.001"/>
+        </geometry>
+      </visual>
+      <collision>
+        <origin xyz="${touchscreen_xyz}" rpy="${touchscreen_rpy}"/>
+        <geometry>
+        <mesh filename="package://kortex_description/meshes/touchscreen.stl" scale="0.001 0.001 0.001"/>
+        </geometry>
+      </collision>
+    </link>
+    <joint name="touchscreen_fixed" type="fixed">
+      <parent link="touchscreen_mount"/>
+      <child  link="touchscreen"/>
+    </joint>
   </xacro:macro>
 </robot>

Commit message: add full body collision for cobot in kortex_description

File: kortex_description/robots/cobot_collision.xacro (robot description, xacro)
@@ -12,7 +12,15 @@
       tower_size:='0.125 0.125 0.306'
       tower_xyz:='0 0 -0.154'
-      touchscreen_mount_xyz:='0.0 -0.065 -0.07'
-      touchscreen_xyz:='-0.15 -0.086 0.06'
-      touchscreen_rpy:='0.78 0 0'">
+      touchscreen_mount_xyz:='-0.065 0 -0.07'
+      touchscreen_xyz:='-0.086 0.15 0.06'
+      touchscreen_rpy:='0.78 0 -1.5708'
+      supporter_460_size:='0.025 0.025 0.46'
+      supporter_460_xyz:='-0.0188 -0.168 -0.06'
+      supporter_580_size:='0.025 0.025 0.58'
+      supporter_580_xyz:='-0.0188 -0.387 0.24'
+      camera_bracket_xyz:='0.001 -0.387 0.497'
+      kinect_xyz:='0.06 -0.387 0.515'
+      kinect_rpy:='1.8326 0 1.5708'
+      ">
     <link name="cobot_base">
       <collision>
@@ -40,12 +48,6 @@
     </joint>
     <link name="touchscreen_mount">
-      <visual>
-        <origin xyz="${touchscreen_mount_xyz}" rpy="0 0 0"/>
-        <geometry>
-        <mesh filename="package://kortex_description/meshes/touchscreen_mount.stl" scale="0.001 0.001 0.001"/>
-        </geometry>
-      </visual>
       <collision>
-        <origin xyz="${touchscreen_mount_xyz}" rpy="0 0 0"/>
+        <origin xyz="${touchscreen_mount_xyz}" rpy="0 0 -1.5708"/>
         <geometry>
         <mesh filename="package://kortex_description/meshes/touchscreen_mount.stl" scale="0.001 0.001 0.001"/>
@@ -58,10 +60,4 @@
     </joint>
     <link name="touchscreen">
-      <visual>
-        <origin xyz="${touchscreen_xyz}" rpy="${touchscreen_rpy}"/>
-        <geometry>
-        <mesh filename="package://kortex_description/meshes/touchscreen.stl" scale="0.001 0.001 0.001"/>
-        </geometry>
-      </visual>
       <collision>
         <origin xyz="${touchscreen_xyz}" rpy="${touchscreen_rpy}"/>
@@ -75,4 +71,52 @@
       <child  link="touchscreen"/>
     </joint>
+    <link name="supporter_460">
+      <collision>
+        <origin xyz="${supporter_460_xyz}" rpy="1.5708 1.5708 0"/>
+        <geometry>
+          <box size="${supporter_460_size}"/>
+        </geometry>
+      </collision>
+    </link>
+    <joint name="supporter_460_fixed" type="fixed">
+      <parent link="cobot_tower"/>
+      <child  link="supporter_460"/>
+    </joint>
+    <link name="supporter_580">
+      <collision>
+        <origin xyz="${supporter_580_xyz}" rpy="0 0 0"/>
+        <geometry>
+          <box size="${supporter_580_size}"/>
+        </geometry>
+      </collision>
+    </link>
+    <joint name="supporter_580_fixed" type="fixed">
+      <parent link="cobot_tower"/>
+      <child  link="supporter_580"/>
+    </joint>
+    <link name="camera_bracket">
+      <collision>
+        <origin xyz="${camera_bracket_xyz}" rpy="0 0 1.5708"/>
+        <geometry>
+        <mesh filename="package://kortex_description/meshes/camera_bracket.stl" scale="0.001 0.001 0.001"/>
+        </geometry>
+      </collision>
+    </link>
+    <joint name="camera_bracket_fixed" type="fixed">
+      <parent link="cobot_tower"/>
+      <child  link="camera_bracket"/>
+    </joint>
+    <link name="kinect">
+      <collision>
+        <origin xyz="${kinect_xyz}" rpy="${kinect_rpy}"/>
+        <geometry>
+        <mesh filename="package://kortex_description/meshes/kinect.stl" scale="0.001 0.001 0.001"/>
+        </geometry>
+      </collision>
+    </link>
+    <joint name="kinect_fixed" type="fixed">
+      <parent link="camera_bracket"/>
+      <child  link="kinect"/>
+    </joint>
   </xacro:macro>
 </robot>

Commit message: finish full body self-collision checking with moveit

File: kortex_description/robots/cobot_collision.xacro (robot description, xacro)
@@ -119,4 +119,18 @@
       <child  link="kinect"/>
     </joint>
+    <link name="kinect_ablated">
+      <collision>
+        <origin xyz="${kinect_xyz}" rpy="${kinect_rpy}"/>
+        <geometry>
+          <!-- <box size="0.11 0.05 0.2"/> -->
+          <!-- alate 4cm -->
+          <box size="0.15 0.09 0.24"/>
+        </geometry>
+      </collision>
+    </link>
+    <joint name="kinect_ablated_fixed" type="fixed">
+      <parent link="camera_bracket"/>
+      <child  link="kinect_ablated"/>
+    </joint>
   </xacro:macro>
 </robot>

Commit message: need kinect to arm base calibration

File: kortex_description/robots/cobot_collision.xacro (robot description, xacro)
@@ -7,4 +7,7 @@
   <xacro:macro name="cobot_collision" params="
       mount_link:=base_link
+      sensor_link:=depth_camera_link
+      sensor_xyz:='0 0 0'
+      sensor_rpy:='0 0 0'
       base_xyz:='0 0 -0.387'
       base_radius:=0.3
@@ -133,4 +136,10 @@
       <child  link="kinect_ablated"/>
     </joint>
+    <link name="${sensor_link}"/>
+    <joint name="$sensor_mount" type="fixed">
+      <parent link="${mount_link}"/>                <!-- or whatever you mount to -->
+      <child  link="${sensor_link}"/>
+      <origin xyz="${sensor_xyz}" rpy="${sensor_rpy}"/>
+    </joint>
   </xacro:macro>
 </robot>

Commit message: fix moveit

File: kortex_description/robots/cobot_collision.xacro (robot description, xacro)
@@ -7,7 +7,4 @@
   <xacro:macro name="cobot_collision" params="
       mount_link:=base_link
-      sensor_link:=depth_camera_link
-      sensor_xyz:='0 0 0'
-      sensor_rpy:='0 0 0'
       base_xyz:='0 0 -0.387'
       base_radius:=0.3
@@ -136,10 +133,4 @@
       <child  link="kinect_ablated"/>
     </joint>
-    <link name="${sensor_link}"/>
-    <joint name="$sensor_mount" type="fixed">
-      <parent link="${mount_link}"/>                <!-- or whatever you mount to -->
-      <child  link="${sensor_link}"/>
-      <origin xyz="${sensor_xyz}" rpy="${sensor_rpy}"/>
-    </joint>
   </xacro:macro>
 </robot>

File: kortex_description/robots/gen3.xacro (robot description, xacro)
@@ -31,12 +31,12 @@
     <xacro:property name="initial_positions_file" default="$(arg initial_positions_file)"/>
     <link name="world" />
-    <link name="/cobot/base_link"/>
+    <!-- <link name="cobot_base_link"/>
     <joint name="world_to_cobot_base" type="fixed">
         <parent link="world"/>
-        <child  link="/cobot/base_link"/>
+        <child  link="cobot_base_link"/>
         <origin xyz="0 0 0" rpy="0 0 0"/>
-    </joint>
+    </joint> -->
     <xacro:load_robot
-        parent="/cobot/base_link"
+        parent="world"
         arm="$(arg arm)"
         gripper="$(arg gripper)"

Commit message: update cobot_collision

File: kortex_description/robots/cobot_collision.xacro (robot description, xacro)
@@ -133,4 +133,28 @@
       <child  link="kinect_ablated"/>
     </joint>
+    <link name="dummy_left_guard">
+      <collision>
+        <origin xyz="0.001 0.8 0.497" rpy="0 0 1.5708"/>
+        <geometry>
+          <box size="0.4 0.4 0.80"/>
+        </geometry>
+      </collision>
+    </link>
+    <joint name="dummy_left_guard_fixed" type="fixed">
+      <parent link="cobot_tower"/>
+      <child  link="dummy_left_guard"/>
+    </joint>
+    <!-- <link name="dummy_front_guard">
+      <collision>
+        <origin xyz="0.8 0.0 -0.4" rpy="0 0 0"/>
+        <geometry>
+          <box size="0.4 0.4 0.1"/>
+        </geometry>
+      </collision>
+    </link>
+    <joint name="dummy_front_guard_fixed" type="fixed">
+      <parent link="cobot_tower"/>
+      <child  link="dummy_front_guard"/>
+    </joint> -->
   </xacro:macro>
 </robot>

Commit message: added obstacle avoidance check

File: kortex_description/robots/cobot_collision.xacro (robot description, xacro)
@@ -24,4 +24,11 @@
       ">
     <link name="cobot_base">
+      <visual>
+        <origin xyz="${base_xyz}" rpy="0 0 0"/>
+        <geometry>
+            <cylinder radius="${base_radius}" length="${base_height}"/>
+        </geometry>
+        <material name="cobot_silver"/>
+      </visual>
       <collision>
         <origin xyz="${base_xyz}" rpy="0 0 0"/>
@@ -36,4 +43,11 @@
     </joint>
     <link name="cobot_tower">
+      <visual>
+        <origin xyz="${tower_xyz}" rpy="0 0 0"/>
+        <geometry>
+          <box size="${tower_size}"/>
+        </geometry>
+        <material name="cobot_silver"/>
+      </visual>
       <collision>
         <origin xyz="${tower_xyz}" rpy="0 0 0"/>
@@ -48,9 +62,16 @@
     </joint>
     <link name="touchscreen_mount">
-      <collision>
+      <visual>
         <origin xyz="${touchscreen_mount_xyz}" rpy="0 0 -1.5708"/>
         <geometry>
         <mesh filename="package://kortex_description/meshes/touchscreen_mount.stl" scale="0.001 0.001 0.001"/>
         </geometry>
+        <material name="cobot_silver"/>
+      </visual>
+      <collision>
+        <origin xyz="${touchscreen_mount_xyz}" rpy="0 0 -1.5708"/>
+        <geometry>
+        <mesh filename="package://kortex_description/meshes/touchscreen_mount.stl" scale="0.001 0.001 0.001"/>
+        </geometry>
       </collision>
     </link>
@@ -60,4 +81,11 @@
     </joint>
     <link name="touchscreen">
+      <visual>
+        <origin xyz="${touchscreen_xyz}" rpy="${touchscreen_rpy}"/>
+        <geometry>
+        <mesh filename="package://kortex_description/meshes/touchscreen.stl" scale="0.001 0.001 0.001"/>
+        </geometry>
+        <material name="cobot_silver"/>
+      </visual>
       <collision>
         <origin xyz="${touchscreen_xyz}" rpy="${touchscreen_rpy}"/>
@@ -72,9 +100,16 @@
     </joint>
     <link name="supporter_460">
-      <collision>
+      <visual>
         <origin xyz="${supporter_460_xyz}" rpy="1.5708 1.5708 0"/>
         <geometry>
           <box size="${supporter_460_size}"/>
         </geometry>
+        <material name="cobot_silver"/>
+      </visual>
+      <collision>
+        <origin xyz="${supporter_460_xyz}" rpy="1.5708 1.5708 0"/>
+        <geometry>
+          <box size="${supporter_460_size}"/>
+        </geometry>
       </collision>
     </link>
@@ -84,9 +119,16 @@
     </joint>
     <link name="supporter_580">
-      <collision>
+      <visual>
         <origin xyz="${supporter_580_xyz}" rpy="0 0 0"/>
         <geometry>
           <box size="${supporter_580_size}"/>
         </geometry>
+        <material name="cobot_silver"/>
+      </visual>
+      <collision>
+        <origin xyz="${supporter_580_xyz}" rpy="0 0 0"/>
+        <geometry>
+          <box size="${supporter_580_size}"/>
+        </geometry>
       </collision>
     </link>
@@ -96,9 +138,16 @@
     </joint>
     <link name="camera_bracket">
-      <collision>
+      <visual>
         <origin xyz="${camera_bracket_xyz}" rpy="0 0 1.5708"/>
         <geometry>
         <mesh filename="package://kortex_description/meshes/camera_bracket.stl" scale="0.001 0.001 0.001"/>
         </geometry>
+        <material name="cobot_silver"/>
+      </visual>
+      <collision>
+        <origin xyz="${camera_bracket_xyz}" rpy="0 0 1.5708"/>
+        <geometry>
+        <mesh filename="package://kortex_description/meshes/camera_bracket.stl" scale="0.001 0.001 0.001"/>
+        </geometry>
       </collision>
     </link>
@@ -108,4 +157,11 @@
     </joint>
     <link name="kinect">
+      <visual>
+        <origin xyz="${kinect_xyz}" rpy="${kinect_rpy}"/>
+        <geometry>
+        <mesh filename="package://kortex_description/meshes/kinect.stl" scale="0.001 0.001 0.001"/>
+        </geometry>
+        <material name="cobot_silver"/>
+      </visual>
       <collision>
         <origin xyz="${kinect_xyz}" rpy="${kinect_rpy}"/>
@@ -120,9 +176,14 @@
     </joint>
     <link name="kinect_ablated">
-      <collision>
-        <origin xyz="${kinect_xyz}" rpy="${kinect_rpy}"/>
-        <geometry>
-          <!-- <box size="0.11 0.05 0.2"/> -->
-          <!-- alate 4cm -->
+      <visual>
+        <origin xyz="${kinect_xyz}" rpy="${kinect_rpy}"/>
+        <geometry>
+          <box size="0.15 0.09 0.24"/>
+        </geometry>
+        <material name="cobot_silver"/>
+      </visual>
+      <collision>
+        <origin xyz="${kinect_xyz}" rpy="${kinect_rpy}"/>
+        <geometry>
           <box size="0.15 0.09 0.24"/>
         </geometry>
@@ -134,4 +195,11 @@
     </joint>
     <link name="dummy_left_guard">
+      <visual>
+        <origin xyz="0.001 0.8 0.497" rpy="0 0 1.5708"/>
+        <geometry>
+          <box size="0.4 0.4 0.80"/>
+        </geometry>
+        <material name="cobot_silver"/>
+      </visual>
       <collision>
         <origin xyz="0.001 0.8 0.497" rpy="0 0 1.5708"/>
