Commit message: xacro

File: kortex_description/robots/cobot_collision.xacro (robot description, xacro)
@@ -198,5 +198,5 @@
         <origin xyz="0.001 0.8 0.497" rpy="0 0 1.5708"/>
         <geometry>
-          <box size="0.4 0.4 0.80"/>
+          <box size="0.5 0.5 0.80"/>
         </geometry>
         <material name="cobot_silver"/>
@@ -205,5 +205,5 @@
         <origin xyz="0.001 0.8 0.497" rpy="0 0 1.5708"/>
         <geometry>
-          <box size="0.4 0.4 0.80"/>
+          <box size="0.5 0.5 0.80"/>
         </geometry>
       </collision>

Commit message: Update Cobot Kinect calibration geometry

File: kortex_description/robots/cobot_collision.xacro (robot description, xacro)
@@ -21,4 +21,5 @@
       camera_bracket_xyz:='0.001 -0.387 0.497'
       kinect_xyz:='0.06 -0.387 0.515'
+      kinect_ablated_xyz:='-0.024 -0.462 0.526'
       kinect_rpy:='1.8326 0 1.5708'
       ">
@@ -177,5 +178,5 @@
     <link name="kinect_ablated">
       <visual>
-        <origin xyz="${kinect_xyz}" rpy="${kinect_rpy}"/>
+        <origin xyz="${kinect_ablated_xyz}" rpy="${kinect_rpy}"/>
         <geometry>
           <box size="0.15 0.09 0.24"/>
@@ -184,5 +185,5 @@
       </visual>
       <collision>
-        <origin xyz="${kinect_xyz}" rpy="${kinect_rpy}"/>
+        <origin xyz="${kinect_ablated_xyz}" rpy="${kinect_rpy}"/>
         <geometry>
           <box size="0.15 0.09 0.24"/>
