Commit message: added optional sensor_3d

File: kortex_description/arms/gen3/7dof/urdf/gen3_macro.xacro (robot description, xacro)
@@ -443,4 +443,19 @@
         xyz="0 0 0" />
     </joint>
+    <link name="${prefix}bracelet_collision_box">
+      <visual>
+        <origin xyz="0.0 -0.05 -0.05" rpy="0 0 0"/>
+        <geometry>
+          <box size="0.12 0.05 0.05"/>
+        </geometry>
+        <material name="">
+          <color rgba="0.700 0.700 0.700 1.000"/>
+        </material>
+      </visual>
+    </link>
+    <joint name="${prefix}bracelet_collision_box_fixed" type="fixed">
+      <parent link="${prefix}bracelet_link"/>
+      <child  link="${prefix}bracelet_collision_box"/>
+    </joint>
     <xacro:if value="${vision}">
       <!-- sim camera needs to be rotated which might not apply to built in vision module -->
